File: CAN-BT_LUT/CAN-BT.brd (EAGLE design)
At the start: 45.1 x 30.5 mm, 30 parts, among them Q1 16MHz, U1 PIC18F25K80, U2 78M05, U3 TJA1055T

Commit message: Small fix
Parts:
- renumbered JP2 to HC-05
Changed lines of the file:
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@@
 <layers>
 <layer number="1" name="Top" color="4" fill="1" visible="yes" active="yes"/>
-<layer number="16" name="Bottom" color="1" fill="1" visible="no" active="yes"/>
+<layer number="16" name="Bottom" color="1" fill="1" visible="yes" active="yes"/>
 <layer number="17" name="Pads" color="2" fill="1" visible="yes" active="yes"/>
 <layer number="18" name="Vias" color="2" fill="1" visible="yes" active="yes"/>
 <layer number="19" name="Unrouted" color="6" fill="1" visible="yes" active="yes"/>
 <layer number="20" name="Dimension" color="15" fill="1" visible="yes" active="yes"/>
-<layer number="21" name="tPlace" color="7" fill="1" visible="yes" active="yes"/>
+<layer number="21" name="tPlace" color="7" fill="1" visible="no" active="yes"/>
 <layer number="22" name="bPlace" color="7" fill="1" visible="no" active="yes"/>
 <layer number="23" name="tOrigins" color="15" fill="1" visible="no" active="yes"/>
 <layer number="24" name="bOrigins" color="15" fill="1" visible="no" active="yes"/>
-<layer number="25" name="tNames" color="7" fill="1" visible="no" active="yes"/>
-<layer number="26" name="bNames" color="7" fill="1" visible="no" active="yes"/>
+<layer number="25" name="tNames" color="7" fill="1" visible="yes" active="yes"/>
+<layer number="26" name="bNames" color="7" fill="1" visible="yes" active="yes"/>
 <layer number="27" name="tValues" color="7" fill="1" visible="no" active="yes"/>
 <layer number="28" name="bValues" color="7" fill="1" visible="no" active="yes"/>
@@
 </element>
 <element name="JP1" library="CAN-BT" package="1X05" value="" x="38.1" y="64.77" rot="MR180"/>
-<element name="JP2" library="CAN-BT" package="1X06" value="" x="62.23" y="52.705" rot="MR90"/>
+<element name="HC-05" library="CAN-BT" package="1X06" value="" x="62.23" y="52.705" rot="MR90"/>
 <element name="LED1" library="CAN-BT" package="LED2X5" value="" x="60.96" y="66.04"/>
 <element name="LED2" library="CAN-BT" package="LED2X5" value="" x="60.96" y="63.5"/>
@@
 <wire x1="52.385" y1="61.275" x2="52.07" y2="60.96" width="0.4064" layer="1"/>
 <contactref element="JP1" pad="3"/>
-<contactref element="JP2" pad="3"/>
+<contactref element="HC-05" pad="3"/>
 <contactref element="LED1" pad="K"/>
 <contactref element="LED2" pad="K"/>
@@
 <wire x1="29.21" y1="58.42" x2="27.94" y2="58.42" width="0.4064" layer="16"/>
 <wire x1="27.94" y1="58.42" x2="27.94" y2="56.99" width="0.4064" layer="16"/>
-<contactref element="JP2" pad="2"/>
+<contactref element="HC-05" pad="2"/>
 <wire x1="58.1025" y1="53.6575" x2="53.0225" y2="53.6575" width="0.4064" layer="1"/>
 <wire x1="53.0225" y1="53.6575" x2="50.8" y2="55.88" width="0.4064" layer="1"/>
@@
 </signal>
 <signal name="EN">
-<contactref element="JP2" pad="1"/>
+<contactref element="HC-05" pad="1"/>
 </signal>
 <signal name="BT_TX">
-<contactref element="JP2" pad="4"/>
+<contactref element="HC-05" pad="4"/>
 <contactref element="U1" pad="18"/>
 <wire x1="55.5625" y1="55.245" x2="53.34" y2="57.4675" width="0.4064" layer="1"/>
@@
 </signal>
 <signal name="BT_RX">
-<contactref element="JP2" pad="5"/>
+<contactref element="HC-05" pad="5"/>
 <contactref element="U1" pad="17"/>
 <wire x1="55.88" y1="56.515" x2="54.61" y2="57.785" width="0.4064" layer="1"/>
@@
 </signal>
 <signal name="STATE">
-<contactref element="JP2" pad="6"/>
+<contactref element="HC-05" pad="6"/>
 <contactref element="R7" pad="2"/>
 <wire x1="59.69" y1="59.0575" x2="62.2275" y2="59.0575" width="0.4064" layer="1"/>
